Commit message: 更改了界面函数，加入了阻抗控制

File: catkin_ws/src/robot_description/armt_description /robots/armt.xacro (robot description, xacro)
@@ -3,5 +3,5 @@
   <xacro:include filename="$(find armt_description)/robots/arm.gazebo" />
   <xacro:include filename="$(find armt_description)/robots/position_transmition.xacro" />
-  <!-- simple  joints macros configure the joint driver and param-->
+  <!-- simple joints macros configure the joint driver and param-->
   <xacro:armt_joint joint_prefix="1"> </xacro:armt_joint>
   <xacro:armt_joint joint_prefix="2"> </xacro:armt_joint>
@@ -11,10 +11,10 @@
   <xacro:armt_joint joint_prefix="6"> </xacro:armt_joint>
   <xacro:armt_joint joint_prefix="7"> </xacro:armt_joint>
-<link name="world"/>
-<joint name="fixed" type="fixed">
-  <parent link="world"/>
-  <child link="base_link"/>
-</joint>
-<link
+  <link name="world"/>
+  <joint name="fixed" type="fixed">
+    <parent link="world"/>
+    <child link="base_link"/>
+  </joint>
+  <link
   name="base_link">
   <inertial>
@@ -38,5 +38,5 @@
     <geometry>
       <mesh
-        filename="package://arm_hand/meshes/base_link.STL" />
+        filename="package://armt_description/meshes/base_link.STL" />
     </geometry>
     <material
@@ -52,5 +52,5 @@
     <geometry>
       <mesh
-        filename="package://arm_hand/meshes/base_link.STL" />
+        filename="package://armt_description/meshes/base_link.STL" />
     </geometry>
   </collision>
@@ -78,5 +78,5 @@
     <geometry>
       <mesh
-        filename="package://arm_hand/meshes/link1.STL" />
+        filename="package://armt_description/meshes/link1.STL" />
     </geometry>
     <material
@@ -92,5 +92,5 @@
     <geometry>
       <mesh
-        filename="package://arm_hand/meshes/link1.STL" />
+        filename="package://armt_description/meshes/link1.STL" />
     </geometry>
   </collision>
@@ -136,5 +136,5 @@
     <geometry>
       <mesh
-        filename="package://arm_hand/meshes/link2.STL" />
+        filename="package://armt_description/meshes/link2.STL" />
     </geometry>
     <material
@@ -150,5 +150,5 @@
     <geometry>
       <mesh
-        filename="package://arm_hand/meshes/link2.STL" />
+        filename="package://armt_description/meshes/link2.STL" />
     </geometry>
   </collision>
@@ -194,5 +194,5 @@
     <geometry>
       <mesh
-        filename="package://arm_hand/meshes/link3.STL" />
+        filename="package://armt_description/meshes/link3.STL" />
     </geometry>
     <material
@@ -208,5 +208,5 @@
     <geometry>
       <mesh
-        filename="package://arm_hand/meshes/link3.STL" />
+        filename="package://armt_description/meshes/link3.STL" />
     </geometry>
   </collision>
@@ -252,5 +252,5 @@
     <geometry>
       <mesh
-        filename="package://arm_hand/meshes/link4.STL" />
+        filename="package://armt_description/meshes/link4.STL" />
     </geometry>
     <material
@@ -266,5 +266,5 @@
     <geometry>
       <mesh
-        filename="package://arm_hand/meshes/link4.STL" />
+        filename="package://armt_description/meshes/link4.STL" />
     </geometry>
   </collision>
@@ -310,5 +310,5 @@
     <geometry>
       <mesh
-        filename="package://arm_hand/meshes/link5.STL" />
+        filename="package://armt_description/meshes/link5.STL" />
     </geometry>
     <material
@@ -324,5 +324,5 @@
     <geometry>
       <mesh
-        filename="package://arm_hand/meshes/link5.STL" />
+        filename="package://armt_description/meshes/link5.STL" />
     </geometry>
   </collision>
@@ -368,5 +368,5 @@
     <geometry>
       <mesh
-        filename="package://arm_hand/meshes/link6.STL" />
+        filename="package://armt_description/meshes/link6.STL" />
     </geometry>
     <material
@@ -382,5 +382,5 @@
     <geometry>
       <mesh
-        filename="package://arm_hand/meshes/link6.STL" />
+        filename="package://armt_description/meshes/link6.STL" />
     </geometry>
   </collision>
@@ -426,5 +426,5 @@
     <geometry>
       <mesh
-        filename="package://arm_hand/meshes/link7.STL" />
+        filename="package://armt_description/meshes/link7.STL" />
     </geometry>
     <material
@@ -440,5 +440,5 @@
     <geometry>
       <mesh
-        filename="package://arm_hand/meshes/link7.STL" />
+        filename="package://armt_description/meshes/link7.STL" />
     </geometry>
   </collision>
@@ -462,3 +462,63 @@
       velocity="2" />
 </joint>
+<link
+  name="sensor_link">
+  <inertial>
+    <origin
+      xyz="0 0 0"
+      rpy="0 0 0" />
+    <mass
+      value="0.10567" />
+    <inertia
+      ixx="7.1441E-05"
+      ixy="1.6499E-08"
+      ixz="-4.9269E-09"
+      iyy="7.146E-05"
+      iyz="-8.5336E-09"
+      izz="0.00013366" />
+  </inertial>
+  <visual>
+    <origin
+      xyz="0 0 0"
+      rpy="0 0 0" />
+    <geometry>
+      <mesh
+        filename="package://armt_description/meshes/sensor_link.STL" />
+    </geometry>
+    <material
+      name="">
+      <color
+        rgba="1 0 0 1" />
+    </material>
+  </visual>
+  <collision>
+    <origin
+      xyz="0 0 0"
+      rpy="0 0 0" />
+    <geometry>
+      <mesh
+        filename="package://armt_description/meshes/sensor_link.STL" />
+    </geometry>
+  </collision>
+</link>
+<joint
+  name="sensor_joint"
+  type="revolute">
+  <origin
+    xyz="0 0 0"
+    rpy="0 0 0.12101" />
+  <parent
+    link="link7" />
+  <child
+    link="sensor_link" />
+  <axis
+    xyz="0 0 1" />
+  <limit
+    lower="0"
+    upper="0"
+    effort="0"
+    velocity="0" />
+  <safety_controller
+    k_velocity="0" />
+</joint>
 </robot>
