Commit message: 主要增加三臂规划

File: catkin_ws/src/robot_description/ur_description/urdf/ur.gazebo.xacro (robot description, xacro)
@@ -16,4 +16,11 @@
     <gazebo reference="${prefix}wrist_3_link">
       <selfCollide>true</selfCollide>
+      <material>Gazebo/Red</material>
+      <mu1 value="1.0"/>
+      <mu2 value="1.0"/>
+      <kp value="10000" />
+      <kd value="1.0" />
+      <fdir1 value="1 0 0"/>
+      <gravity value="true"/>
     </gazebo>
     <gazebo reference="${prefix}wrist_2_link">
