Commit message: 增加了手抓

File: catkin_ws/src/robot_description/armc_description/robot/armc1.xacro (robot description, xacro)
@@ -509,5 +509,5 @@
     <origin
       xyz="0 0 0.192"
-      rpy="0 0 0.12101" />
+      rpy="0 -0.025 0.0" />
     <parent
       link="Link7" />

File: catkin_ws/src/robot_description/armc_description/urdf/armc_description.urdf (robot description, URDF)
Before this commit: robot armc_description, 10 links, 9 joints
Joints:
- joint sensor_joint: type revolute -> fixed
