Commit message: 2020年9月23号

File: catkin_ws/src/robot_description/armc_description/robot/armc.xacro (robot description, xacro)
@@ -457,4 +457,62 @@
       xyz="0 0 1" />
     <limit
+      lower="-10"
+      upper="10"
+      effort="20"
+      velocity="20" />
+  </joint>
+  <link
+    name="sensor_link">
+    <inertial>
+      <origin
+        xyz="5.187E-06 8.9595E-06 0.011516"
+        rpy="0 0 0" />
+      <mass
+        value="0.10567" />
+      <inertia
+        ixx="7.1441E-05"
+        ixy="1.6499E-08"
+        ixz="-4.9269E-09"
+        iyy="7.146E-05"
+        iyz="-8.5336E-09"
+        izz="0.00013366" />
+    </inertial>
+    <visual>
+      <origin
+        xyz="0 0 0"
+        rpy="0 0 0" />
+      <geometry>
+        <mesh
+          filename="package://armc_description/meshes/sensor_link.STL" />
+      </geometry>
+      <material
+        name="">
+        <color
+          rgba="1 0 0 1" />
+      </material>
+    </visual>
+    <collision>
+      <origin
+        xyz="0 0 0"
+        rpy="0 0 0" />
+      <geometry>
+        <mesh
+          filename="package://armc_description/meshes/sensor_link.STL" />
+      </geometry>
+    </collision>
+  </link>
+  <joint
+    name="sensor_joint"
+    type="revolute">
+    <origin
+      xyz="0 0 0.192"
+      rpy="0 0 0.12101" />
+    <parent
+      link="Link7" />
+    <child
+      link="sensor_link" />
+    <axis
+      xyz="0 0 1" />
+    <limit
       lower="0"
       upper="0"
@@ -464,63 +522,3 @@
       k_velocity="0" />
   </joint>
-  <link
-    name="sensor_link">
-    <inertial>
-      <origin
-        xyz="5.187E-06 8.9595E-06 0.011516"
-        rpy="0 0 0" />
-      <mass
-        value="0.10567" />
-      <inertia
-        ixx="7.1441E-05"
-        ixy="1.6499E-08"
-        ixz="-4.9269E-09"
-        iyy="7.146E-05"
-        iyz="-8.5336E-09"
-        izz="0.00013366" />
-    </inertial>
-    <visual>
-      <origin
-        xyz="0 0 0"
-        rpy="0 0 0" />
-      <geometry>
-        <mesh
-          filename="package://armc_description/meshes/sensor_link.STL" />
-      </geometry>
-      <material
-        name="">
-        <color
-          rgba="1 0 0 1" />
-      </material>
-    </visual>
-    <collision>
-      <origin
-        xyz="0 0 0"
-        rpy="0 0 0" />
-      <geometry>
-        <mesh
-          filename="package://armc_description/meshes/sensor_link.STL" />
-      </geometry>
-    </collision>
-  </link>
-  <joint
-    name="sensor_joint"
-    type="revolute">
-    <origin
-      xyz="0 0 0.192"
-      rpy="0 0 0.12101" />
-    <parent
-      link="Link7" />
-    <child
-      link="sensor_link" />
-    <axis
-      xyz="0 0 1" />
-    <limit
-      lower="0"
-      upper="0"
-      effort="0"
-      velocity="0" />
-    <safety_controller
-      k_velocity="0" />
-  </joint>
 </robot>

File: catkin_ws/src/robot_description/armc_description/robot/armc1.xacro (robot description, xacro)
@@ -457,4 +457,64 @@
       xyz="0 0 1" />
     <limit
+      lower="-10"
+      upper="10"
+      effort="20"
+      velocity="20" />
+    <safety_controller
+      k_velocity="1" />
+  </joint>
+  <link
+    name="sensor_link">
+    <inertial>
+      <origin
+        xyz="5.187E-06 8.9595E-06 0.011516"
+        rpy="0 0 0" />
+      <mass
+        value="0.10567" />
+      <inertia
+        ixx="7.1441E-05"
+        ixy="1.6499E-08"
+        ixz="-4.9269E-09"
+        iyy="7.146E-05"
+        iyz="-8.5336E-09"
+        izz="0.00013366" />
+    </inertial>
+    <visual>
+      <origin
+        xyz="0 0 0"
+        rpy="0 0 0" />
+      <geometry>
+        <mesh
+          filename="package://armc_description/meshes/sensor_link.STL" />
+      </geometry>
+      <material
+        name="">
+        <color
+          rgba="1 0 0 1" />
+      </material>
+    </visual>
+    <collision>
+      <origin
+        xyz="0 0 0"
+        rpy="0 0 0" />
+      <geometry>
+        <mesh
+          filename="package://armc_description/meshes/sensor_link.STL" />
+      </geometry>
+    </collision>
+  </link>
+  <joint
+    name="sensor_joint"
+    type="revolute">
+    <origin
+      xyz="0 0 0.192"
+      rpy="0 -0.025 0.0" />
+    <parent
+      link="Link7" />
+    <child
+      link="sensor_link" />
+    <axis
+      xyz="0 0 1" />
+    <limit
       lower="0"
       upper="0"
@@ -464,64 +524,4 @@
       k_velocity="0" />
   </joint>
-  <link
-    name="sensor_link">
-    <inertial>
-      <origin
-        xyz="5.187E-06 8.9595E-06 0.011516"
-        rpy="0 0 0" />
-      <mass
-        value="0.10567" />
-      <inertia
-        ixx="7.1441E-05"
-        ixy="1.6499E-08"
-        ixz="-4.9269E-09"
-        iyy="7.146E-05"
-        iyz="-8.5336E-09"
-        izz="0.00013366" />
-    </inertial>
-    <visual>
-      <origin
-        xyz="0 0 0"
-        rpy="0 0 0" />
-      <geometry>
-        <mesh
-          filename="package://armc_description/meshes/sensor_link.STL" />
-      </geometry>
-      <material
-        name="">
-        <color
-          rgba="1 0 0 1" />
-      </material>
-    </visual>
-    <collision>
-      <origin
-        xyz="0 0 0"
-        rpy="0 0 0" />
-      <geometry>
-        <mesh
-          filename="package://armc_description/meshes/sensor_link.STL" />
-      </geometry>
-    </collision>
-  </link>
-  <joint
-    name="sensor_joint"
-    type="revolute">
-    <origin
-      xyz="0 0 0.192"
-      rpy="0 -0.025 0.0" />
-    <parent
-      link="Link7" />
-    <child
-      link="sensor_link" />
-    <axis
-      xyz="0 0 1" />
-    <limit
-      lower="0"
-      upper="0"
-      effort="0"
-      velocity="0" />
-    <safety_controller
-      k_velocity="0" />
-  </joint>
     <link
     name="actuator">

File: catkin_ws/src/robot_description/armc_description/robot_finger/armc.xacro (robot description, xacro)
@@ -517,10 +517,10 @@
       xyz="0 0 1" />
     <limit
-      lower="0"
-      upper="0"
-      effort="0"
-      velocity="0" />
+      lower="-10"
+      upper="10"
+      effort="10"
+      velocity="10" />
     <safety_controller
-      k_velocity="0" />
+      k_velocity="1" />
   </joint>
  <link
