Commit message: 增加了三臂打磨框架

File: catkin_ws/src/robot_description/finger/urdf/finger.urdf (robot description, URDF)
Before this commit: robot finger, 2 links, 1 joints
Links:
- added link world
Joints:
- added joint fixed: type fixed, parent world, child base_link

File: catkin_ws/src/robot_description/ur_description/urdf/ur.gazebo.xacro (robot description, xacro)
@@ -19,5 +19,5 @@
       <mu1 value="1.0"/>
       <mu2 value="1.0"/>
-      <kp value="10000" />
+      <kp value="100000" />
       <kd value="1.0" />
       <fdir1 value="1 0 0"/>
