Commit message: 误删

File: catkin_ws/src/robot_description/armc_description/robot_finger/armc.xacro (robot description, xacro)
@@ -524,9 +524,9 @@
       k_velocity="0" />
   </joint>
-  <link
+ <link
     name="finger_Link1">
     <inertial>
       <origin
-        xyz="0 0 0"
+        xyz="0.0014547 -2.6021E-18 0.030405"
         rpy="0 0 0" />
       <mass
@@ -534,8 +534,8 @@
       <inertia
         ixx="0.00023035"
-        ixy="-3.7311E-21"
+        ixy="-2.7465E-21"
         ixz="-3.4957E-05"
         iyy="0.00033399"
-        iyz="-1.4134E-20"
+        iyz="-1.2385E-20"
         izz="0.00025833" />
     </inertial>
@@ -564,23 +564,10 @@
     </collision>
   </link>
-  <joint
-    name="fixed_joint"
-    type="fixed">
-    <origin
-      xyz="0 0 0.023"
+  <joint name="fixed1" type="fixed">
+  <origin
+      xyz="-0 0 0.024"
       rpy="0 0 0" />
-    <parent
-      link="sensor_link" />
-    <child
-      link="finger_Link1" />
-    <axis
-      xyz="0 0 1" />
-    <limit
-      lower="0"
-      upper="0"
-      effort="0"
-      velocity="0" />
-    <safety_controller
-      k_velocity="0" />
+    <parent link="sensor_link"/>
+    <child link="finger_Link1"/>
   </joint>
   <link
@@ -588,5 +575,5 @@
     <inertial>
       <origin
-        xyz="-0.01025 6.9389E-18 0.064"
+        xyz="-0.0045141 1.1276E-17 0.024"
         rpy="0 0 0" />
       <mass
@@ -594,8 +581,8 @@
       <inertia
         ixx="4.604E-05"
-        ixy="-1.175E-21"
+        ixy="-1.1647E-21"
         ixz="-8.085E-06"
         iyy="4.6086E-05"
-        iyz="-4.3195E-21"
+        iyz="-4.3089E-21"
         izz="9.0463E-06" />
     </inertial>
@@ -628,5 +615,5 @@
     type="prismatic">
     <origin
-      xyz="0 0 0"
+      xyz="-0.0057359 0 0.04"
       rpy="0 0 0" />
     <parent
@@ -638,7 +625,7 @@
     <limit
       lower="0"
-      upper="-10"
+      upper="0.05"
       effort="100"
-      velocity="60" />
+      velocity="100" />
   </joint>
 </robot>

File: catkin_ws/src/robot_description/finger/urdf/finger.urdf (robot description, URDF)
Before this commit: robot finger, 3 links, 2 joints
Links:
- removed link finger_Link2
- removed link world
- added link finger_Link, mass 0.06; collision mesh filename=package://finger/meshes/finger_Link.STL; visual mesh filename=package://finger/meshes/finger_Link.STL
Joints:
- removed joint finger_joint
- removed joint fixed
- added joint hand_joint: type prismatic, parent base_link, child finger_Link, origin xyz=-0.0057359 0 0.04 rpy=0 0 0, axis -1 0 0, limit lower=0 upper=0.05 effort=100 velocity=100
