Commit message: 解决了armt的1关节反馈问题

File: catkin_ws/src/robot_description/ur_description/robot_hand/ur.gazebo.xacro (robot description, xacro)
@@ -31,4 +31,21 @@
     <gazebo reference="${prefix}sensor_link">
       <selfCollide>true</selfCollide>
+      <material>Gazebo/Red</material>
+      <mu1 value="1.0"/>
+      <mu2 value="1.0"/>
+      <kp value="100000" />
+      <kd value="1.0" />
+      <fdir1 value="1 0 0"/>
+      <gravity value="true"/>
+    </gazebo>
+     <gazebo reference="${prefix}finger_Link2">
+      <selfCollide>true</selfCollide>
+      <material>Gazebo/Red</material>
+      <mu1 value="1.0"/>
+      <mu2 value="1.0"/>
+      <kp value="100000" />
+      <kd value="1.0" />
+      <fdir1 value="1 0 0"/>
+      <gravity value="true"/>
     </gazebo>
     </gazebo>
